Commit message: navigation successful with basic robot

File: catkin_ws/src/udacity_bot/urdf/udacity_bot.xacro (robot description, xacro)
@@ -135,5 +135,5 @@
             <origin xyz="-0.15 0 -0.05" rpy=" 0 0 0"/>
             <geometry>
-                <sphere radius="0.05"/>
+                <sphere radius="0.0499"/>
 				        <material name="green"/>
             </geometry>
@@ -159,5 +159,5 @@
             <origin xyz="0.15 0 -0.05" rpy=" 0 0 0"/>
             <geometry>
-                <sphere radius="0.05"/>
+                <sphere radius="0.0499"/>
             </geometry>
             <surface>

Commit message: AMCL not converging, but robot designed

File: catkin_ws/src/udacity_bot/urdf/udacity_bot.xacro (robot description, xacro)
@@ -10,5 +10,5 @@
     <link name='left_wheel'>
         <inertial>
-            <mass value="5.0"/>
+            <mass value="3.0"/>
             <origin xyz="0.0 0 0" rpy=" 0 1.5707 1.5707"/>
             <inertia ixx="0.1" ixy="0" ixz="0" iyy="0.1" iyz="0" izz="0.1"/>
@@ -23,5 +23,5 @@
             <origin xyz="0.0 0 0" rpy=" 0 1.5707 1.5707"/>
             <geometry>
-                <cylinder length="0.05" radius="0.1"/>
+                <cylinder length="0.025" radius="0.1"/>
             </geometry>
 			      <material name="black"/>
@@ -29,5 +29,5 @@
     </link>
     <joint type="continuous" name="left_wheel_hinge">
-        <origin xyz="0.0 0.25 0" rpy="0 0 0"/>
+        <origin xyz="0.10 0.14 0" rpy="0 0 0"/>
         <child link="left_wheel"/>
         <parent link="chassis"/>
@@ -38,5 +38,5 @@
     <link name='right_wheel'>
         <inertial>
-            <mass value="5.0"/>
+            <mass value="3.0"/>
             <origin xyz="0.0 0 0" rpy=" 0 1.5707 1.5707"/>
             <inertia ixx="0.1" ixy="0" ixz="0" iyy="0.1" iyz="0" izz="0.1"/>
@@ -45,5 +45,5 @@
             <origin xyz="0.0 0 0" rpy=" 0 1.5707 1.5707"/>
             <geometry>
-                <cylinder length="0.05" radius="0.1"/>
+                <cylinder length="0.025" radius="0.1"/>
             </geometry>
         </collision>
@@ -51,5 +51,5 @@
             <origin xyz="0.0 0 0" rpy=" 0 1.5707 1.5707"/>
             <geometry>
-                <cylinder length="0.05" radius="0.1"/>
+                <cylinder length="0.025" radius="0.1"/>
             </geometry>
 			      <material name="black"/>
@@ -57,5 +57,5 @@
     </link>
     <joint type="continuous" name="right_wheel_hinge">
-        <origin xyz="0 -0.25 0" rpy="0 0 0"/>
+        <origin xyz="0.10 -0.14 0" rpy="0 0 0"/>
         <child link="right_wheel"/>
         <parent link="chassis"/>
@@ -84,5 +84,5 @@
     </link>
     <joint type="fixed" name="camera_joint">
-        <origin xyz="0.2 0 0" rpy="0 0 0"/>
+        <origin xyz="0.16 0 0" rpy="0 0 0"/>
         <child link="camera"/>
         <parent link="chassis"/>
@@ -108,5 +108,5 @@
     </link>
     <joint type="fixed" name="hokuyo_joint">
-        <origin xyz="0.175 0.0 0.1" rpy="0 0 0"/>
+        <origin xyz="0.125 0.0 0.1" rpy="0 0 0"/>
         <child link="hokuyo"/>
         <parent link="chassis"/>
@@ -115,5 +115,5 @@
         <pose>0 0 0.1 0 0 0</pose>
         <inertial>
-            <mass value="15.0"/>
+            <mass value="5.0"/>
             <origin xyz="0.0 0 0" rpy=" 0 0 0"/>
             <inertia ixx="0.1" ixy="0" ixz="0" iyy="0.1" iyz="0" izz="0.1"/>
@@ -122,5 +122,5 @@
             <origin xyz="0 0 0" rpy=" 0 0 0"/>
             <geometry>
-                <box size=".4 .4 .1"/>
+                <box size=".3 .2 .1"/>
             </geometry>
         </collision>
@@ -128,5 +128,5 @@
             <origin xyz="0 0 0" rpy=" 0 0 0"/>
             <geometry>
-                <box size=".4 .4 .1"/>
+                <box size=".3 .2 .1"/>
             </geometry>
 			      <material name="blue"/>
@@ -135,5 +135,5 @@
             <origin xyz="-0.15 0 -0.05" rpy=" 0 0 0"/>
             <geometry>
-                <sphere radius="0.0499"/>
+                <sphere radius="0.0495"/>
 				        <material name="green"/>
             </geometry>
@@ -150,5 +150,5 @@
         </collision>
         <visual name='back_caster_visual'>
-            <origin xyz="-0.15 0 -0.05" rpy=" 0 0 0"/>
+            <origin xyz="-0.1 0 -0.05" rpy=" 0 0 0"/>
             <geometry>
                 <sphere radius="0.05"/>
@@ -156,4 +156,5 @@
             </geometry>
         </visual>
+<!--
         <collision name='front_caster_collision'>
             <origin xyz="0.15 0 -0.05" rpy=" 0 0 0"/>
@@ -179,4 +180,5 @@
             </geometry>
         </visual>
+-->
     </link>
 </robot>

Commit message: New robot not reaching the goal. Unsure why

File: catkin_ws/src/udacity_bot/urdf/udacity_bot.xacro (robot description, xacro)
@@ -29,9 +29,9 @@
     </link>
     <joint type="continuous" name="left_wheel_hinge">
-        <origin xyz="0.10 0.14 0" rpy="0 0 0"/>
+        <origin xyz="0.0 0.14 0" rpy="0 0 0"/>
         <child link="left_wheel"/>
         <parent link="chassis"/>
         <axis xyz="0 1 0" rpy="0 0 0"/>
-        <limit effort="10000" velocity="1000"/>
+        <limit effort="2500" velocity="250"/>
         <joint_properties damping="1.0" friction="1.0"/>
     </joint>
@@ -57,9 +57,9 @@
     </link>
     <joint type="continuous" name="right_wheel_hinge">
-        <origin xyz="0.10 -0.14 0" rpy="0 0 0"/>
+        <origin xyz="0.0 -0.14 0" rpy="0 0 0"/>
         <child link="right_wheel"/>
         <parent link="chassis"/>
         <axis xyz="0 1 0" rpy="0 0 0"/>
-        <limit effort="10000" velocity="1000"/>
+        <limit effort="2500" velocity="250"/>
         <joint_properties damping="1.0" friction="1.0"/>
     </joint>
@@ -135,5 +135,5 @@
             <origin xyz="-0.15 0 -0.05" rpy=" 0 0 0"/>
             <geometry>
-                <sphere radius="0.0495"/>
+                <sphere radius="0.0499"/>
 				        <material name="green"/>
             </geometry>
@@ -156,5 +156,4 @@
             </geometry>
         </visual>
-<!--
         <collision name='front_caster_collision'>
             <origin xyz="0.15 0 -0.05" rpy=" 0 0 0"/>
@@ -180,5 +179,4 @@
             </geometry>
         </visual>
--->
     </link>
 </robot>

Commit message: r2d2 robot successfully reaches the goal

File: catkin_ws/src/udacity_bot/urdf/udacity_bot.xacro (robot description, xacro)
@@ -17,21 +17,21 @@
             <origin xyz="0.0 0 0" rpy=" 0 1.5707 1.5707"/>
             <geometry>
+                <cylinder length="0.049" radius="0.1"/>
+            </geometry>
+        </collision>
+        <visual name='wheel_visual'>
+            <origin xyz="0.0 0 0" rpy=" 0 1.5707 1.5707"/>
+            <geometry>
                 <cylinder length="0.05" radius="0.1"/>
             </geometry>
-        </collision>
-        <visual name='wheel_visual'>
-            <origin xyz="0.0 0 0" rpy=" 0 1.5707 1.5707"/>
-            <geometry>
-                <cylinder length="0.025" radius="0.1"/>
-            </geometry>
 			      <material name="black"/>
         </visual>
     </link>
     <joint type="continuous" name="left_wheel_hinge">
-        <origin xyz="0.0 0.14 0" rpy="0 0 0"/>
+        <origin xyz="0.0 0.225 -0.15" rpy="0 0 0"/>
         <child link="left_wheel"/>
         <parent link="chassis"/>
         <axis xyz="0 1 0" rpy="0 0 0"/>
-        <limit effort="2500" velocity="250"/>
+        <limit effort="25000" velocity="250"/>
         <joint_properties damping="1.0" friction="1.0"/>
     </joint>
@@ -45,5 +45,5 @@
             <origin xyz="0.0 0 0" rpy=" 0 1.5707 1.5707"/>
             <geometry>
-                <cylinder length="0.025" radius="0.1"/>
+                <cylinder length="0.049" radius="0.1"/>
             </geometry>
         </collision>
@@ -51,5 +51,5 @@
             <origin xyz="0.0 0 0" rpy=" 0 1.5707 1.5707"/>
             <geometry>
-                <cylinder length="0.025" radius="0.1"/>
+                <cylinder length="0.05" radius="0.1"/>
             </geometry>
 			      <material name="black"/>
@@ -57,9 +57,9 @@
     </link>
     <joint type="continuous" name="right_wheel_hinge">
-        <origin xyz="0.0 -0.14 0" rpy="0 0 0"/>
+        <origin xyz="0.0 -0.225 -0.15" rpy="0 0 0"/>
         <child link="right_wheel"/>
         <parent link="chassis"/>
         <axis xyz="0 1 0" rpy="0 0 0"/>
-        <limit effort="2500" velocity="250"/>
+        <limit effort="25000" velocity="250"/>
         <joint_properties damping="1.0" friction="1.0"/>
     </joint>
@@ -84,5 +84,5 @@
     </link>
     <joint type="fixed" name="camera_joint">
-        <origin xyz="0.16 0 0" rpy="0 0 0"/>
+        <origin xyz="0.2 0 0" rpy="0 0 0"/>
         <child link="camera"/>
         <parent link="chassis"/>
@@ -108,30 +108,54 @@
     </link>
     <joint type="fixed" name="hokuyo_joint">
-        <origin xyz="0.125 0.0 0.1" rpy="0 0 0"/>
+        <origin xyz="0.0 0.0 0.2" rpy="0 0 0"/>
         <child link="hokuyo"/>
-        <parent link="chassis"/>
+        <parent link="head"/>
     </joint>
     <link name='chassis'>
         <pose>0 0 0.1 0 0 0</pose>
-        <inertial>
-            <mass value="5.0"/>
-            <origin xyz="0.0 0 0" rpy=" 0 0 0"/>
-            <inertia ixx="0.1" ixy="0" ixz="0" iyy="0.1" iyz="0" izz="0.1"/>
-        </inertial>
-        <collision name='collision'>
-            <origin xyz="0 0 0" rpy=" 0 0 0"/>
-            <geometry>
-                <box size=".3 .2 .1"/>
-            </geometry>
+        <collision name='collision'>
+          <origin xyz="0.0 0 0.0" rpy="0 0 0"/>
+          <geometry>
+              <cylinder length="0.3" radius="0.2"/>
+          </geometry>
         </collision>
         <visual name='chassis_visual'>
-            <origin xyz="0 0 0" rpy=" 0 0 0"/>
-            <geometry>
-                <box size=".3 .2 .1"/>
-            </geometry>
+          <origin xyz="0.0 0 0" rpy=" 0 0 0"/>
+          <geometry>
+              <cylinder length="0.4" radius="0.2"/>
+          </geometry>
 			      <material name="blue"/>
         </visual>
+        <visual name='back_caster_visual'>
+            <origin xyz="-0.145 0 -0.2" rpy=" 0 0 0"/>
+            <geometry>
+                <sphere radius="0.05"/>
+                <material name="green"/>
+            </geometry>
+        </visual>
         <collision name='back_caster_collision'>
-            <origin xyz="-0.15 0 -0.05" rpy=" 0 0 0"/>
+            <origin xyz="-0.145 0 -0.2" rpy=" 0 0 0"/>
+            <geometry>
+                <sphere radius="0.0499"/>
+            </geometry>
+            <surface>
+                <friction>
+                    <ode>
+                        <mu>0</mu>
+                        <mu2>0</mu2>
+                        <slip1>1.0</slip1>
+                        <slip2>1.0</slip2>
+                    </ode>
+                </friction>
+            </surface>
+        </collision>
+        <visual name='back_left_caster_visual'>
+            <origin xyz="-0.1 -0.1 -0.2" rpy=" 0 0 0"/>
+            <geometry>
+                <sphere radius="0.05"/>
+            </geometry>
+        </visual>
+        <collision name='back_left_caster_collision'>
+            <origin xyz="-0.1 -0.1 -0.2" rpy=" 0 0 0"/>
             <geometry>
                 <sphere radius="0.0499"/>
@@ -149,6 +173,44 @@
             </surface>
         </collision>
-        <visual name='back_caster_visual'>
-            <origin xyz="-0.1 0 -0.05" rpy=" 0 0 0"/>
+        <visual name='back_right_caster_visual'>
+            <origin xyz="-0.1 0.1 -0.2" rpy=" 0 0 0"/>
+            <geometry>
+                <sphere radius="0.05"/>
+            </geometry>
+        </visual>
+        <collision name='back_right_caster_collision'>
+            <origin xyz="-0.1 0.1 -0.2" rpy=" 0 0 0"/>
+            <geometry>
+                <sphere radius="0.0499"/>
+            </geometry>
+            <surface>
+                <friction>
+                    <ode>
+                        <mu>0</mu>
+                        <mu2>0</mu2>
+                        <slip1>1.0</slip1>
+                        <slip2>1.0</slip2>
+                    </ode>
+                </friction>
+            </surface>
+        </collision>
+        <collision name='front_caster_collision'>
+            <origin xyz="0.145 0 -0.2" rpy=" 0 0 0"/>
+            <geometry>
+                <sphere radius="0.0499"/>
+            </geometry>
+            <surface>
+                <friction>
+                    <ode>
+                        <mu>0</mu>
+                        <mu2>0</mu2>
+                        <slip1>1.0</slip1>
+                        <slip2>1.0</slip2>
+                    </ode>
+                </friction>
+            </surface>
+        </collision>
+        <visual name='front_caster_visual'>
+            <origin xyz="0.145 0 -0.2" rpy=" 0 0 0"/>
             <geometry>
                 <sphere radius="0.05"/>
@@ -156,27 +218,79 @@
             </geometry>
         </visual>
-        <collision name='front_caster_collision'>
-            <origin xyz="0.15 0 -0.05" rpy=" 0 0 0"/>
-            <geometry>
-                <sphere radius="0.0499"/>
-            </geometry>
-            <surface>
-                <friction>
-                    <ode>
-                        <mu>0</mu>
-                        <mu2>0</mu2>
-                        <slip1>1.0</slip1>
-                        <slip2>1.0</slip2>
-                    </ode>
-                </friction>
-            </surface>
-        </collision>
-        <visual name='front_caster_visual'>
-            <origin xyz="0.15 0 -0.05" rpy=" 0 0 0"/>
-            <geometry>
-                <sphere radius="0.05"/>
-				        <material name="green"/>
-            </geometry>
-        </visual>
-    </link>
+        <visual name='front_right_caster_visual'>
+            <origin xyz="0.1 0.1 -0.2" rpy=" 0 0 0"/>
+            <geometry>
+                <sphere radius="0.05"/>
+            </geometry>
+        </visual>
+        <collision name='front_right_caster_collision'>
+            <origin xyz="0.1 0.1 -0.2" rpy=" 0 0 0"/>
+            <geometry>
+                <sphere radius="0.0499"/>
+            </geometry>
+            <surface>
+                <friction>
+                    <ode>
+                        <mu>0</mu>
+                        <mu2>0</mu2>
+                        <slip1>1.0</slip1>
+                        <slip2>1.0</slip2>
+                    </ode>
+                </friction>
+            </surface>
+        </collision>
+        <visual name='front_left_caster_visual'>
+            <origin xyz="-0.1 -0.1 -0.2" rpy=" 0 0 0"/>
+            <geometry>
+                <sphere radius="0.05"/>
+            </geometry>
+        </visual>
+        <collision name='front_left_caster_collision'>
+            <origin xyz="0.1 -0.1 -0.2" rpy=" 0 0 0"/>
+            <geometry>
+                <sphere radius="0.0499"/>
+            </geometry>
+            <surface>
+                <friction>
+                    <ode>
+                        <mu>0</mu>
+                        <mu2>0</mu2>
+                        <slip1>1.0</slip1>
+                        <slip2>1.0</slip2>
+                    </ode>
+                </friction>
+            </surface>
+        </collision>
+    </link>
+    <link name='head'>
+      <visual>
+        <geometry>
+          <sphere radius='0.2'/>
+        </geometry>
+        <material name='white'/>
+      </visual>
+    </link>
+    <joint name='head_joint' type='fixed'>
+      <parent link='chassis'/>
+      <child link='head'/>
+      <origin xyz='0 0 0.2'/>
+    </joint>
+    <link name='ballast'>
+      <inertial>
+          <mass value="5.0"/>
+          <origin xyz="0 0 0" rpy="0 0 0"/>
+          <inertia ixx="0.1" ixy="0" ixz="0" iyy="0.1" iyz="0" izz="0.1"/>
+      </inertial>
+      <visual>
+        <geometry>
+          <box size='0.01 0.01 0.1'/>
+        </geometry>
+        <material name='white'/>
+      </visual>
+    </link>
+    <joint name='ballast_joint' type='fixed'>
+      <parent link='chassis'/>
+      <child link='ballast'/>
+      <origin xyz='0 0 0.05'/>
+    </joint>
 </robot>
